Commit message: Modificacoes no modelo mais o controlador projetado

File: tilt/robots/model.urdf (robot description, URDF)
Before this commit: robot tilt, 6 links, 5 joints
Links:
- link corpo: mass 1.908310289141 -> 1.92834614495378
- link helicedir: mass 0.00963319741474509 -> 0.00963033406162666
- link heliceesq: mass 0.00963319729836474 -> 0.00963022071477903
- link servodir: mass 0.0713136390603168 -> 0.0709329033977977
- link servoesq: mass 0.0713136390866666 -> 0.071313642110537
Joints:
- removed joint thrustdir
- removed joint thrustesq
- added joint thurstdir: type continuous, parent servodir, child helicedir, origin xyz=0 0 0 rpy=0 0 1.35525271560688E-20, axis 0 0 1
- added joint thurstesq: type continuous, parent servoesq, child heliceesq, origin xyz=0 0 0 rpy=3.46944695195361E-18 -3.46944695195361E-18 -1.0842021724855E-19, axis 0 0 1
- joint aL: axis -0.000108446791897333 0.999999994119647 0 -> 0 0.999999999985527 0; limit lower=-1 upper=1 effort=10 velocity=10 -> lower=-6 upper=6 effort=10 velocity=10; origin xyz=0.000774317061806635 0.277601419719204 0.0549353011331433 rpy=0.0264243899580086 -0.000142465393102244 -0.000108408934057588 -> xyz=-0.00355649276858555 0.278215496595548 0.100523302768374 rpy=0.0261844653212001 -0.0185928637494992 -0.000483121778388988
- joint aR: axis -9.98351002423385E-05 -0.999999995016477 0 -> 0 -0.999999999985527 0; limit lower=-1 upper=1 effort=10 velocity=10 -> lower=-6 upper=6 effort=10 velocity=10; origin xyz=-1.8271804286945E-05 -0.277611425055307 0.0549286993075094 rpy=-0.0261799241453877 0.000147944076641961 9.98008905062241E-05 -> xyz=-0.00434908257730353 -0.277007353402455 0.100523186479296 rpy=-0.0261800852026307 -0.0033472956926336 9.14579673019161E-05
